File: board/electrospinner-pcb/electrospinner.sch (KiCad schematic (older format))
At the start: 42 parts, among them SW1 ResetBTN, U1 FT230XS, U2 A4988SETTR-T, U3 MSP430G2553IPW20

Commit message: Adds all footprints
Parts:
- C10, C11, C14, C8, C9: footprint (none) -> Capacitor_SMD:C_0603_1608Metric
- C12, C5, C6: footprint (none) -> Capacitor_SMD:C_0805_2012Metric
- SW1: footprint (none) -> Button_Switch_SMD:SW_SPST_EVPBF
Changed lines of the file:
@@
 F 0 "C6" H 2000 2900 50  0000 L CNN
 F 1 "3.3uF" H 1950 2800 50  0000 L CNN
-F 2 "" H 1900 2900 50  0001 C CNN
+F 2 "Capacitor_SMD:C_0805_2012Metric" H 1900 2900 50  0001 C CNN
 F 3 "~" H 1900 2900 50  0001 C CNN
 	1    1900 2900
@@
 F 0 "C5" H 2000 1600 50  0000 L CNN
 F 1 "3.3uF" H 2000 1500 50  0000 L CNN
-F 2 "" H 1900 1600 50  0001 C CNN
+F 2 "Capacitor_SMD:C_0805_2012Metric" H 1900 1600 50  0001 C CNN
 F 3 "~" H 1900 1600 50  0001 C CNN
 	1    1900 1600
@@
 F 0 "SW1" V 4496 1702 50  0000 R CNN
 F 1 "ResetBTN" V 4405 1702 50  0000 R CNN
-F 2 "" H 4450 1950 50  0001 C CNN
+F 2 "Button_Switch_SMD:SW_SPST_EVPBF" H 4450 1950 50  0001 C CNN
 F 3 "" H 4450 1950 50  0001 C CNN
 	1    4450 1750
@@
 F 0 "C9" V 4800 5500 50  0000 C CNN
 F 1 "0.1uF" V 4800 5700 50  0000 C CNN
-F 2 "" H 4800 6000 50  0001 C CNN
+F 2 "Capacitor_SMD:C_0603_1608Metric" H 4800 6000 50  0001 C CNN
 F 3 "~" H 4800 6000 50  0001 C CNN
 	1    4800 6000
@@
 F 0 "C11" H 5200 6600 50  0000 L CNN
 F 1 "0.22uF" H 5100 6500 50  0000 L CNN
-F 2 "" H 5400 6650 50  0001 C CNN
+F 2 "Capacitor_SMD:C_0603_1608Metric" H 5400 6650 50  0001 C CNN
 F 3 "~" H 5400 6650 50  0001 C CNN
 	1    5400 6650
@@
 F 0 "C10" H 5100 3700 50  0000 L CNN
 F 1 "0.1uF" H 5050 3600 50  0000 L CNN
-F 2 "" H 5350 3650 50  0001 C CNN
+F 2 "Capacitor_SMD:C_0603_1608Metric" H 5350 3650 50  0001 C CNN
 F 3 "~" H 5350 3650 50  0001 C CNN
 	1    5350 3650
@@
 F 0 "C14" H 5842 3696 50  0000 L CNN
 F 1 "0.1uF" H 5842 3605 50  0000 L CNN
-F 2 "" H 5750 3650 50  0001 C CNN
+F 2 "Capacitor_SMD:C_0603_1608Metric" H 5750 3650 50  0001 C CNN
 F 3 "~" H 5750 3650 50  0001 C CNN
 	1    5750 3650
@@
 F 0 "C12" H 5550 4050 50  0000 L CNN
 F 1 "1uF" H 5550 3950 50  0000 L CNN
-F 2 "" H 5450 4050 50  0001 C CNN
-F 3 "~" H 5450 4050 50  0001 C CNN
+F 2 "Capacitor_SMD:C_0805_2012Metric" H 5450 4050 50  0001 C CNN
+F 3 "http://www.samsungsem.com/kr/support/product-search/mlcc/CL10B104KB8NNNC.jsp" H 5450 4050 50  0001 C CNN
 	1    5450 4050
 	1    0    0    -1
@@
 F 0 "C8" V 4271 4450 50  0000 C CNN
 F 1 "0.1uF" V 4362 4450 50  0000 C CNN
-F 2 "" H 4500 4450 50  0001 C CNN
+F 2 "Capacitor_SMD:C_0603_1608Metric" H 4500 4450 50  0001 C CNN
 F 3 "~" H 4500 4450 50  0001 C CNN
 	1    4500 4450

Commit message: Removes sense resistors from stepper driver
Parts:
- removed R10, R11: ?k, Resistor_SMD:R_0201_0603Metric, symbol Device:R_Small_US
Connections:
- wire segments 204 -> 200
- no-connect marks 8 -> 10
Other:
- moved on the sheet: 5Vin1
Changed lines of the file:
@@
 L electrospinner-rescue:Barrel_Jack_MountingPin-Connector-electrospinner-rescue 5Vin1
 U 1 1 5C8B25DD
-P 750 1850
-F 0 "5Vin1" H 650 2200 50  0000 C CNN
-F 1 "BarrelJack" H 600 2100 50  0000 C CNN
-F 2 "Connector_BarrelJack:BarrelJack_Horizontal" H 800 1810 50  0001 C CNN
-F 3 "~" H 800 1810 50  0001 C CNN
-	1    750  1850
+P 850 2000
+F 0 "5Vin1" H 750 2350 50  0000 C CNN
+F 1 "BarrelJack" H 700 2250 50  0000 C CNN
+F 2 "Connector_BarrelJack:BarrelJack_Horizontal" H 900 1960 50  0001 C CNN
+F 3 "~" H 900 1960 50  0001 C CNN
+	1    850  2000
 	1    0    0    -1
 $EndComp
@@
 L power:GNDD #PWR0102
 U 1 1 5C8C5B3B
-P 1100 2150
-F 0 "#PWR0102" H 1100 1900 50  0001 C CNN
-F 1 "GNDD" H 1104 1995 50  0001 C CNN
-F 2 "" H 1100 2150 50  0001 C CNN
-F 3 "" H 1100 2150 50  0001 C CNN
-	1    1100 2150
+P 1200 2300
+F 0 "#PWR0102" H 1200 2050 50  0001 C CNN
+F 1 "GNDD" H 1204 2145 50  0001 C CNN
+F 2 "" H 1200 2300 50  0001 C CNN
+F 3 "" H 1200 2300 50  0001 C CNN
+	1    1200 2300
 	1    0    0    -1
 $EndComp
@@
 L power:GNDD #PWR0103
 U 1 1 5C8C5B75
-P 750 2150
-F 0 "#PWR0103" H 750 1900 50  0001 C CNN
-F 1 "GNDD" H 754 1995 50  0001 C CNN
-F 2 "" H 750 2150 50  0001 C CNN
-F 3 "" H 750 2150 50  0001 C CNN
-	1    750  2150
+P 850 2300
+F 0 "#PWR0103" H 850 2050 50  0001 C CNN
+F 1 "GNDD" H 854 2145 50  0001 C CNN
+F 2 "" H 850 2300 50  0001 C CNN
+F 3 "" H 850 2300 50  0001 C CNN
+	1    850  2300
 	1    0    0    -1
 $EndComp
@@
 L power:+5V #PWR0111
 U 1 1 5C8DC2DB
-P 1100 1650
-F 0 "#PWR0111" H 1100 1500 50  0001 C CNN
-F 1 "+5V" H 1115 1823 50  0000 C CNN
-F 2 "" H 1100 1650 50  0001 C CNN
-F 3 "" H 1100 1650 50  0001 C CNN
-	1    1100 1650
+P 1200 1800
+F 0 "#PWR0111" H 1200 1650 50  0001 C CNN
+F 1 "+5V" H 1215 1973 50  0000 C CNN
+F 2 "" H 1200 1800 50  0001 C CNN
+F 3 "" H 1200 1800 50  0001 C CNN
+	1    1200 1800
 	1    0    0    -1
 $EndComp
@@
 $EndComp
 Wire Wire Line
-	1050 1750 1100 1750
-Wire Wire Line
-	1100 1750 1100 1650
-Wire Wire Line
-	1100 1950 1050 1950
-Wire Wire Line
-	1100 1950 1100 2150
+	1150 1900 1200 1900
+Wire Wire Line
+	1200 1900 1200 1800
+Wire Wire Line
+	1200 2100 1150 2100
+Wire Wire Line
+	1200 2100 1200 2300
 $Comp
 L Motor:Stepper_Motor_unipolar_6pin StepperMotor1
@@
 $EndComp
 Wire Wire Line
-	5650 6500 5650 6650
-$Comp
-L Device:R_Small_US R10
-U 1 1 5CCE3EFD
-P 5650 6750
-F 0 "R10" H 5500 6800 50  0000 L CNN
-F 1 "?k" H 5500 6700 50  0000 L CNN
-F 2 "Resistor_SMD:R_0201_0603Metric" H 5650 6750 50  0001 C CNN
-F 3 "~" H 5650 6750 50  0001 C CNN
-	1    5650 6750
-	1    0    0    -1
-$EndComp
-Wire Wire Line
-	5750 6500 5750 6650
-$Comp
-L Device:R_Small_US R11
-U 1 1 5CCEBA1D
-P 5750 6750
-F 0 "R11" H 5818 6796 50  0000 L CNN
-F 1 "?k" H 5818 6705 50  0000 L CNN
-F 2 "Resistor_SMD:R_0201_0603Metric" H 5750 6750 50  0001 C CNN
-F 3 "~" H 5750 6750 50  0001 C CNN
-	1    5750 6750
-	1    0    0    -1
-$EndComp
-Wire Wire Line
-	5650 6850 5650 6900
-$Comp
-L power:GNDD #PWR0133
-U 1 1 5CCEBAA9
-P 5650 6900
-F 0 "#PWR0133" H 5650 6650 50  0001 C CNN
-F 1 "GNDD" H 5654 6745 50  0001 C CNN
-F 2 "" H 5650 6900 50  0001 C CNN
-F 3 "" H 5650 6900 50  0001 C CNN
-	1    5650 6900
-	1    0    0    -1
-$EndComp
-Wire Wire Line
-	5750 6850 5750 6900
-$Comp
-L power:GNDD #PWR0134
-U 1 1 5CCF3117
-P 5750 6900
-F 0 "#PWR0134" H 5750 6650 50  0001 C CNN
-F 1 "GNDD" H 5754 6745 50  0001 C CNN
-F 2 "" H 5750 6900 50  0001 C CNN
-F 3 "" H 5750 6900 50  0001 C CNN
-	1    5750 6900
-	1    0    0    -1
-$EndComp
-Wire Wire Line
 	5350 6500 5250 6500
 Wire Wire Line
@@
 Wire Wire Line
 	4200 3600 4400 3600
+NoConn ~ 5650 6500
+NoConn ~ 5750 6500
 $EndSCHEMATC

Commit message: Updates footprints, adds bom
Parts:
- Barrel_Jack1: renamed from 5Vin1; MPN (none) -> 474-PRT-00119
- C1: renamed from C2; MPN (none) -> 80-T529P106M06AAE200
- C10, C14, C8, C9: MPN (none) -> C0805X104K4RACAUTO
- C11: MPN (none) -> 08055C224K4T4A
- C12: MPN (none) -> CL10B104KB8NNNC
- C13, C7: MPN (none) -> 80-T529P106M06AAE200
- C2: renamed from C1; MPN (none) -> 80-T529P106M06AAE200
- C3: renamed from C5; MPN (none) -> 810-CGA4J1X8L335K125
- C4: renamed from C6; MPN (none) -> 810-CGA4J1X8L335K125
- C5: renamed from C4; MPN (none) -> CL21A226KQCLRNC
- C6: renamed from C3; MPN (none) -> CL21A226KQCLRNC
- L1: renamed from L2; footprint Inductor_SMD:L_Wuerth_MAPI-2510 -> Inductor_SMD:L_0805_2012Metric; MPN (none) -> DFE201612PD-1R0M=P2
- L2: renamed from L1; footprint Inductor_SMD:L_Wuerth_MAPI-2510 -> Inductor_SMD:L_0805_2012Metric; MPN (none) -> DFE201612PD-1R0M=P2
- Pt1: renamed from Pt1000; MPN (none) -> 0900766b815bb283; Manufacturer (none) -> Emea
- R1: renamed from R3; value 471k -> 470k; footprint Resistor_SMD:R_0201_0603Metric -> Resistor_SMD:R_0805_2012Metric; MPN (none) -> AC0805FR-10470KL
- R2: renamed from R4; footprint Resistor_SMD:R_0201_0603Metric -> Resistor_SMD:R_0805_2012Metric; MPN (none) -> AC0805FR-13100KL
- R3: renamed from R1; footprint Resistor_SMD:R_0201_0603Metric -> Resistor_SMD:R_0805_2012Metric; MPN (none) -> ERJ-6RED5603V
- R4: renamed from R2; footprint Resistor_SMD:R_0201_0603Metric -> Resistor_SMD:R_0805_2012Metric; MPN (none) -> CRCW0805150KFKEAC
- R5, R6: footprint Resistor_SMD:R_0201_0603Metric -> Resistor_SMD:R_0805_2012Metric; MPN (none) -> ERJ-6RBD3900V
- R7: footprint Resistor_SMD:R_0201_0603Metric -> Resistor_SMD:R_0805_2012Metric; MPN (none) -> MSP430G2553IPW20
- R8: renamed from R12; footprint Resistor_SMD:R_1210_3225Metric -> Resistor_SMD:R_0805_2012Metric; MPN (none) -> RT0805FRE07158RL
- SW1: footprint Button_Switch_SMD:SW_SPST_EVPBF -> Button_Switch_THT:SW_PUSH_6mm_H5mm
- U1: MPN (none) -> FT230XS-R
- U2: renamed from 5V_to_4V1; MPN (none) -> TPS62147RGXR
- U3: renamed from 5V_to_3V3; MPN (none) -> TPS62147RGXR
- USB_B_Header1: value USB_B -> USB_B_Header?
- renumbered MotorConnector_Male1 to MotorConnector_Female1, MotorConnector_Male2 to MotorConnector_Male1, U2 to U4, U3 to U5

Commit message: Updates BOM and footprints, adds spreadsheet
Parts:
- Barrel_Jack1: MPN 474-PRT-00119 -> PRT-00119
- C1, C13, C2, C7: MPN 80-T529P106M06AAE200 -> C0805X106K8RACAUTO
- C10, C11, C14, C8, C9: footprint Capacitor_SMD:C_0603_1608Metric -> Capacitor_SMD:C_0805_2012Metric
- C12: MPN CL10B104KB8NNNC -> C0805C105Z5VACTU
- C3, C4: MPN 810-CGA4J1X8L335K125 -> CGA4J1X8L1C335K125AC
- C5, C6: value 2uF -> 2.2uF; MPN CL21A226KQCLRNC -> 08056C225KAT2A
- D1, D2, MotorConnector_Female1, MotorConnector_Male1, SW1, Temp_Female1, Temp_Male1, USB_B_Header1: Status (none) -> resource-center
- Pt1, StepperMotor1, U1: Status (none) -> ordered
- R7: MPN MSP430G2553IPW20 -> SG73G2ATTD1001D
- U2, U3: Status (none) -> oredered
- U4: Status Active -> ordered
- U5: MPN (none) -> MSP430G2553IPW20; Status (none) -> ordered
Changed lines of the file:
@@
 F 4 "0900766b815bb283" H 0   0   50  0001 C CNN "MPN"
 F 5 "Emea" H 0   0   50  0001 C CNN "Manufacturer"
+F 6 "ordered" H 0   0   50  0001 C CNN "Status"
 	1    10450 1050
 	1    0    0    -1
@@
 F 2 "Connector_USB:USB_B_OST_USB-B1HSxx_Horizontal" H 1600 6750 50  0001 C CNN
 F 3 " ~" H 1600 6750 50  0001 C CNN
+F 4 "resource-center" H 0   0   50  0001 C CNN "Status"
 	1    1450 6800
 	1    0    0    -1
@@
 F 2 "Connector_BarrelJack:BarrelJack_Horizontal" H 900 1960 50  0001 C CNN
 F 3 "~" H 900 1960 50  0001 C CNN
-F 4 " 474-PRT-00119 " H 0   0   50  0001 C CNN "MPN"
+F 4 " PRT-00119 " H 0   0   50  0001 C CNN "MPN"
 	1    850  2000
 	1    0    0    -1
@@
 F 3 "http://www.ti.com/lit/gpn/tps62147" H 2350 550 50  0001 C CNN
 F 4 "TPS62147RGXR" H 0   0   50  0001 C CNN "MPN"
+F 5 "oredered" H 0   0   50  0001 C CNN "Status"
 	1    2350 550
 	1    0    0    -1
@@
 F 2 "Package_SO:TSSOP-20_4.4x6.5mm_P0.65mm" H 5250 1900 50  0001 C CIN
 F 3 "http://www.ti.com/lit/ds/symlink/msp430g2553.pdf" H 6650 2450 50  0001 C CNN
+F 4 "MSP430G2553IPW20" H 0   0   50  0001 C CNN "MPN"
+F 5 "ordered" H 0   0   50  0001 C CNN "Status"
 	1    6700 2450
 	1    0    0    -1
@@
 F 1 "10uF" H 1350 1350 50  0000 L CNN
 F 2 "Capacitor_SMD:C_0805_2012Metric" H 1600 1400 50  0001 C CNN
-F 3 "https://www.mouser.com/datasheet/2/212/T520D108M2R5ATE006-1265335-1488592.pdf" H 1600 1400 50  0001 C CNN
-F 4 "80-T529P106M06AAE200" H 0   0   50  0001 C CNN "MPN"
+F 3 "https://www.mouser.com/datasheet/2/212/KEM_C1078_X7R_FT-CAP_AUTO_SMD-1103315.pdf" H 1600 1400 50  0001 C CNN
+F 4 "C0805X106K8RACAUTO" H 0   0   50  0001 C CNN "MPN"
 	1    1600 1400
 	1    0    0    -1
@@
 P 3600 1200
 F 0 "C5" H 3692 1246 50  0000 L CNN
-F 1 "2uF" H 3692 1155 50  0000 L CNN
+F 1 "2.2uF" H 3692 1155 50  0000 L CNN
 F 2 "Capacitor_SMD:C_0805_2012Metric" H 3600 1200 50  0001 C CNN
-F 3 "http://www.samsungsem.com/kr/support/product-search/mlcc/CL21A226KQCLRNC.jsp" H 3600 1200 50  0001 C CNN
-F 4 "CL21A226KQCLRNC" H 0   0   50  0001 C CNN "MPN"
+F 3 "https://www.mouser.com/datasheet/2/40/X7RDielectric-777024.pdf" H 3600 1200 50  0001 C CNN
+F 4 "08056C225KAT2A" H 0   0   50  0001 C CNN "MPN"
 F 5 "" H 0   0   50  0001 C CNN "Manufacturer"
 	1    3600 1200
@@
 F 3 "http://www.ti.com/lit/gpn/tps62147" H 2350 1850 50  0001 C CNN
 F 4 "TPS62147RGXR" H 0   0   50  0001 C CNN "MPN"
+F 5 "oredered" H 0   0   50  0001 C CNN "Status"
 	1    2350 1850
 	1    0    0    -1
@@
 F 1 "10uF" H 1350 2650 50  0000 L CNN
 F 2 "Capacitor_SMD:C_0805_2012Metric" H 1600 2700 50  0001 C CNN
-F 3 "https://www.mouser.com/datasheet/2/212/T520D108M2R5ATE006-1265335-1488592.pdf" H 1600 2700 50  0001 C CNN
-F 4 "80-T529P106M06AAE200" H 0   0   50  0001 C CNN "MPN"
+F 3 "https://www.mouser.com/datasheet/2/212/KEM_C1078_X7R_FT-CAP_AUTO_SMD-1103315.pdf" H 1600 2700 50  0001 C CNN
+F 4 "C0805X106K8RACAUTO" H 0   0   50  0001 C CNN "MPN"
 	1    1600 2700
 	1    0    0    -1
@@
 P 3600 2500
 F 0 "C6" H 3692 2546 50  0000 L CNN
-F 1 "2uF" H 3692 2455 50  0000 L CNN
+F 1 "2.2uF" H 3692 2455 50  0000 L CNN
 F 2 "Capacitor_SMD:C_0805_2012Metric" H 3600 2500 50  0001 C CNN
-F 3 "http://www.samsungsem.com/kr/support/product-search/mlcc/CL21A226KQCLRNC.jsp" H 3600 2500 50  0001 C CNN
-F 4 "CL21A226KQCLRNC" H 0   0   50  0001 C CNN "MPN"
+F 3 "https://www.mouser.com/datasheet/2/40/X7RDielectric-777024.pdf" H 3600 2500 50  0001 C CNN
+F 4 "08056C225KAT2A" H 0   0   50  0001 C CNN "MPN"
 F 5 "" H 0   0   50  0001 C CNN "Manufacturer"
 	1    3600 2500
@@
 F 2 "LED_SMD:LED_0603_1608Metric" V 3150 5350 50  0001 C CNN
 F 3 "~" V 3150 5350 50  0001 C CNN
+F 4 "resource-center" H 0   0   50  0001 C CNN "Status"
 	1    3150 5350
 	1    0    0    -1
@@
 F 2 "LED_SMD:LED_0603_1608Metric" V 3150 5450 50  0001 C CNN
 F 3 "~" V 3150 5450 50  0001 C CNN
+F 4 "resource-center" H 0   0   50  0001 C CNN "Status"
 	1    3150 5450
 	1    0    0    -1
@@
 F 3 "http://www.ftdichip.com/Products/ICs/FT230X.html" H 2050 5150 50  0001 C CNN
 F 4 "FT230XS-R" H 0   0   50  0001 C CNN "MPN"
+F 5 "ordered" H 0   0   50  0001 C CNN "Status"
 	1    2050 5150
 	1    0    0    -1
@@
 F 2 "" H 8560 5490 50  0001 C CNN
 F 3 "" H 8560 5490 50  0001 C CNN
+F 4 "ordered" H 0   0   50  0001 C CNN "Status"
 	1    8550 5500
 	1    0    0    -1
@@
 F 2 "Connector_JST:JST_EH_B02B-EH-A_1x06_P2.50mm_Vertical" H 7200 5400 50  0001 C CNN
 F 3 "~" H 7200 5400 50  0001 C CNN
+F 4 "resource-center" H 0   0   50  0001 C CNN "Status"
 	1    7200 5400
 	1    0    0    -1
@@
 F 2 "" H 7500 5400 50  0001 C CNN
 F 3 "~" H 7500 5400 50  0001 C CNN
+F 4 "resource-center" H 0   0   50  0001 C CNN "Status"
 	1    7500 5400
 	1    0    0    -1
@@
 F 2 "Connector_JST:JST_EH_B02B-EH-A_1x02_P2.50mm_Vertical" H 9350 1000 50  0001 C CNN
 F 3 "~" H 9350 1000 50  0001 C CNN
+F 4 "resource-center" H 0   0   50  0001 C CNN "Status"
 	1    9350 1000
 	1    0    0    -1
@@
 F 2 "" H 9800 1000 50  0001 C CNN
 F 3 "~" H 9800 1000 50  0001 C CNN
+F 4 "resource-center" H 0   0   50  0001 C CNN "Status"
 	1    9800 1000
 	1    0    0    -1
@@
 F 2 "Capacitor_SMD:C_0805_2012Metric" H 1900 2900 50  0001 C CNN
 F 3 "https://www.mouser.com/datasheet/2/400/lcc_automotive_general_en-843974.pdf" H 1900 2900 50  0001 C CNN
-F 4 "810-CGA4J1X8L335K125" H 0   0   50  0001 C CNN "MPN"
+F 4 "CGA4J1X8L1C335K125AC" H 0   0   50  0001 C CNN "MPN"
 	1    1900 2900
 	1    0    0    -1
@@
 F 2 "Capacitor_SMD:C_0805_2012Metric" H 1900 1600 50  0001 C CNN
 F 3 "https://www.mouser.com/datasheet/2/400/lcc_automotive_general_en-843974.pdf" H 1900 1600 50  0001 C CNN
-F 4 "810-CGA4J1X8L335K125" H 0   0   50  0001 C CNN "MPN"
+F 4 "CGA4J1X8L1C335K125AC" H 0   0   50  0001 C CNN "MPN"
 	1    1900 1600
 	1    0    0    -1
@@
 F 1 "1k" H 4300 2100 50  0000 L CNN
 F 2 "Resistor_SMD:R_0805_2012Metric" H 4450 2100 50  0001 C CNN
-F 3 "https://www.mouser.com/datasheet/2/447/PYu-SR_D_F_tol_RoHS_L_3-1488676.pdf" H 4450 2100 50  0001 C CNN
-F 4 "MSP430G2553IPW20" H 0   0   50  0001 C CNN "MPN"
+F 3 "https://www.mouser.com/datasheet/2/219/SG73G-1316861.pdf" H 4450 2100 50  0001 C CNN
+F 4 " SG73G2ATTD1001D " H 0   0   50  0001 C CNN "MPN"
 	1    4450 2100
 	1    0    0    -1
@@
 F 2 "Button_Switch_THT:SW_PUSH_6mm_H5mm" H 4450 1950 50  0001 C CNN
 F 3 "" H 4450 1950 50  0001 C CNN
+F 4 "resource-center" H 0   0   50  0001 C CNN "Status"
 	1    4450 1750
 	0    -1   -1   0
@@
 F 10 "IC MTR DRVR BIPOLAR 3-5.5V 28QFN" H 5750 6500 60  0001 L CNN "Description"
 F 11 "Allegro MicroSystems, LLC" H 5750 6600 60  0001 L CNN "Manufacturer"
-F 12 "Active" H 5750 6700 60  0001 L CNN "Status"
+F 12 "ordered" H 5750 6700 60  0001 L CNN "Status"
 	1    5550 5500
 	1    0    0    -1
@@
 F 0 "C9" V 4800 5500 50  0000 C CNN
 F 1 "0.1uF" V 4800 5700 50  0000 C CNN
-F 2 "Capacitor_SMD:C_0603_1608Metric" H 4800 6000 50  0001 C CNN
+F 2 "Capacitor_SMD:C_0805_2012Metric" H 4800 6000 50  0001 C CNN
 F 3 "https://www.mouser.com/datasheet/2/212/KEM_C1078_X7R_FT-CAP_AUTO_SMD-1103315.pdf" H 4800 6000 50  0001 C CNN
 F 4 "C0805X104K4RACAUTO" H 0   0   50  0001 C CNN "MPN"
@@
 F 0 "C11" H 5200 6600 50  0000 L CNN
 F 1 "0.22uF" H 5100 6500 50  0000 L CNN
-F 2 "Capacitor_SMD:C_0603_1608Metric" H 5400 6650 50  0001 C CNN
+F 2 "Capacitor_SMD:C_0805_2012Metric" H 5400 6650 50  0001 C CNN
 F 3 "https://www.mouser.com/datasheet/2/40/AutoMLCC-777028.pdf" H 5400 6650 50  0001 C CNN
 F 4 "08055C224K4T4A" H 0   0   50  0001 C CNN "MPN"
@@
 F 1 "10uF" H 5550 3550 50  0000 L CNN
 F 2 "Capacitor_SMD:C_0805_2012Metric" H 5550 3650 50  0001 C CNN
-F 3 "https://www.mouser.com/datasheet/2/212/T520D108M2R5ATE006-1265335-1488592.pdf" H 5550 3650 50  0001 C CNN
-F 4 "80-T529P106M06AAE200" H 0   0   50  0001 C CNN "MPN"
+F 3 "https://www.mouser.com/datasheet/2/212/KEM_C1078_X7R_FT-CAP_AUTO_SMD-1103315.pdf" H 5550 3650 50  0001 C CNN
+F 4 "C0805X106K8RACAUTO" H 0   0   50  0001 C CNN "MPN"
 	1    5550 3650
 	1    0    0    -1
@@
 F 0 "C10" H 5100 3700 50  0000 L CNN
 F 1 "0.1uF" H 5050 3600 50  0000 L CNN
-F 2 "Capacitor_SMD:C_0603_1608Metric" H 5350 3650 50  0001 C CNN
+F 2 "Capacitor_SMD:C_0805_2012Metric" H 5350 3650 50  0001 C CNN
 F 3 "https://www.mouser.com/datasheet/2/212/KEM_C1078_X7R_FT-CAP_AUTO_SMD-1103315.pdf" H 5350 3650 50  0001 C CNN
 F 4 "C0805X104K4RACAUTO" H 0   0   50  0001 C CNN "MPN"
@@
 F 0 "C14" H 5842 3696 50  0000 L CNN
 F 1 "0.1uF" H 5842 3605 50  0000 L CNN
-F 2 "Capacitor_SMD:C_0603_1608Metric" H 5750 3650 50  0001 C CNN
+F 2 "Capacitor_SMD:C_0805_2012Metric" H 5750 3650 50  0001 C CNN
 F 3 "https://www.mouser.com/datasheet/2/212/KEM_C1078_X7R_FT-CAP_AUTO_SMD-1103315.pdf" H 5750 3650 50  0001 C CNN
 F 4 "C0805X104K4RACAUTO" H 0   0   50  0001 C CNN "MPN"
@@
 F 2 "Capacitor_SMD:C_0805_2012Metric" H 5450 4050 50  0001 C CNN
 F 3 "http://www.samsungsem.com/kr/support/product-search/mlcc/CL10B104KB8NNNC.jsp" H 5450 4050 50  0001 C CNN
-F 4 "CL10B104KB8NNNC" H 0   0   50  0001 C CNN "MPN"
+F 4 "C0805C105Z5VACTU" H 0   0   50  0001 C CNN "MPN"
 	1    5450 4050
 	1    0    0    -1
@@
 F 1 "10uF" V 4637 4100 50  0000 C CNN
 F 2 "Capacitor_SMD:C_0805_2012Metric" H 4500 4100 50  0001 C CNN
-F 3 "https://www.mouser.com/datasheet/2/212/T520D108M2R5ATE006-1265335-1488592.pdf" H 4500 4100 50  0001 C CNN
-F 4 "80-T529P106M06AAE200" H 0   0   50  0001 C CNN "MPN"
+F 3 "https://www.mouser.com/datasheet/2/212/KEM_C1078_X7R_FT-CAP_AUTO_SMD-1103315.pdf" H 4500 4100 50  0001 C CNN
+F 4 "C0805X106K8RACAUTO" H 0   0   50  0001 C CNN "MPN"
 	1    4500 4100
 	0    -1   -1   0
@@
 F 0 "C8" V 4271 4450 50  0000 C CNN
 F 1 "0.1uF" V 4362 4450 50  0000 C CNN
-F 2 "Capacitor_SMD:C_0603_1608Metric" H 4500 4450 50  0001 C CNN
+F 2 "Capacitor_SMD:C_0805_2012Metric" H 4500 4450 50  0001 C CNN
 F 3 "https://www.mouser.com/datasheet/2/212/KEM_C1078_X7R_FT-CAP_AUTO_SMD-1103315.pdf" H 4500 4450 50  0001 C CNN
 F 4 "C0805X104K4RACAUTO" H 0   0   50  0001 C CNN "MPN"

Commit message: Saves schematic rev 1
Parts:
- added J?: Header_02x02, Connector_PinHeader_1.00mm:PinHeader_2x02_P1.00mm_Vertical, symbol Connector_Generic:Conn_02x02_Counter_Clockwise
Connections:
- net labels added: DVCC, DVSS, TEST
- wire segments 200 -> 204
Other:
- moved on the sheet: C10, C11, C12, C13, C14, C7, C8, C9, MotorConnector_Female1, MotorConnector_Male1, StepperMotor1

Commit message: Half-done finishing v2 of schematic
Parts:
- removed C10, C14, C8, C9: 0.1uF, Capacitor_SMD:C_0805_2012Metric, symbol Device:C_Small
- removed C11: 0.22uF, Capacitor_SMD:C_0805_2012Metric, symbol Device:C_Small
- removed C12: 1uF, Capacitor_SMD:C_0805_2012Metric, symbol Device:C_Small
- removed C13, C7: 10uF, Capacitor_SMD:C_0805_2012Metric, symbol Device:CP1_Small
- removed U4: A4988SETTR-T, digikey-footprints:VFQFN-28-1EP_5x5mm, symbol dk_PMIC-Motor-Drivers-Controllers:A4988SETTR-T
- added A?: Pololu_Breakout_A4988-Driver_Motor, Module:Pololu_Breakout-16_15.2x20.3mm, symbol electrospinner-rescue:Pololu_Breakout_A4988-Driver_Motor-electrospinner-rescue
- added C? (x3): 0.1uF, symbol Device:C_Small
- added C?: C_Small, symbol Device:C_Small
- added C?: 100uF, symbol Device:CP1_Small
- U1: symbol Interface_USB:FT230XS -> electrospinner-rescue:FT230XS-Interface_USB
- gave numbers to parts that had none: 1
Connections:
- net labels added: +12V, MOTOR_DIR, MOTOR_MS1, MOTOR_MS2, MOTOR_MS3, MOTOR_STEP, ~MOTOR_ENABLE, ~MOTOR_RESET, ~MOTOR_SLEEP
- net labels removed: REF, ROSC, VBB1, VBB2, VCP, VDD, ~MotorRESET
- wire segments 204 -> 183
- no-connect marks 10 -> 8
Other:
- moved on the sheet: R7
