File: board/electrospinner-pcb/electrospinner.sch (KiCad schematic (older format))
At the start: 34 parts, among them J1 Header_02x02, SW1 ResetBTN, U1 FT230XS, U3 TPS62147, U5 MSP430G2553IPW20

Commit message: Updates board to rev 3
Updates thematic
Updates bom
Parts:
- removed A1: A4988_Breakout, Module:Pololu_Breakout-16_15.2x20.3mm, symbol electrospinner-rescue:Pololu_Breakout_A4988-Driver_Motor-electrospinner-rescue
- added A1: Pololu_Breakout_DRV8825, Module:Pololu_Breakout-16_15.2x20.3mm, symbol Driver_Motor:Pololu_Breakout_DRV8825
- added C11: 0.1uF, symbol electrospinner-rescue:C_Small-Device
- USB_B_Header1: value USB_B_Header? -> USB
Connections:
- net labels added: MotorMS#, MotorSLEEP, ~MotorFLT, ~MotorRESET, ~MotorRST
- net labels removed: MOTOR_DIR, MOTOR_MS1, MOTOR_MS2, MOTOR_MS3, MOTOR_STEP, ~MOTOR_ENABLE, ~MOTOR_RESET, ~MOTOR_SLEEP
- wire segments 166 -> 171
Other:
- moved on the sheet: C1, C2, C3
