File: board/electrospinner-pcb/electrospinner.sch (KiCad schematic (older format))
At the start: 35 parts, among them J1 Header_02x02, SW1 ResetBTN, U1 FT230XS, U3 TPS62147, U5 MSP430G2553IPW20

Commit message: Updates to rev5
Parts:
- removed Barrel_Jack1: BarrelJack, Connector_BarrelJack:BarrelJack_Horizontal, symbol electrospinner-rescue:Barrel_Jack_MountingPin-Connector-electrospinner-rescue
- removed C10: 0.1uF, Capacitor_SMD:C_0603_1608Metric, symbol electrospinner-rescue:C_Small-Device
- removed C11: 0.1uF, symbol electrospinner-rescue:C_Small-Device
- removed C5: 0.1uF, Capacitor_SMD:C_0603_1608Metric, symbol Device:C_Small
- removed MotorConnector_Male1: JST_1x6_Male, symbol electrospinner-rescue:Conn_01x06_Male-Connector
- removed Pt1: RS Pro 2371607, symbol electrospinner-rescue:Thermistor_PTC-Device-electrospinner-rescue
- removed R2: 100, Resistor_SMD:R_0805_2012Metric, symbol Device:R_Small_US
- removed StepperMotor1: SY42STH47-1206A, symbol electrospinner-rescue:Stepper_Motor_unipolar_6pin-Motor
- removed Temp_Male1: JST_1x2_Male, symbol electrospinner-rescue:Conn_01x02_Male-Connector
- added C4, C6: 0.1uF, Capacitor_SMD:C_0805_2012Metric, symbol Device:C_Small
- added J1: 12Vin, Connector_BarrelJack:BarrelJack_CUI_PJ-063AH_Horizontal, symbol Connector:Barrel_Jack_MountingPin
- added TP1: ~MotorRST, TestPoint:TestPoint_Keystone_5015_Micro-Minature, symbol Connector:TestPoint
- added TP10: MotorM2, TestPoint:TestPoint_Keystone_5015_Micro-Minature, symbol Connector:TestPoint
- added TP11: MotorSTEP, TestPoint:TestPoint_Keystone_5015_Micro-Minature, symbol Connector:TestPoint
- added TP2: ~MotorEN, TestPoint:TestPoint_Keystone_5015_Micro-Minature, symbol Connector:TestPoint
- added TP3: ~MotorSLP, TestPoint:TestPoint_Keystone_5015_Micro-Minature, symbol Connector:TestPoint
- added TP4: MotorDIR, TestPoint:TestPoint_Keystone_5015_Micro-Minature, symbol Connector:TestPoint
- added TP5: ~MotorFLT, TestPoint:TestPoint_Keystone_5015_Micro-Minature, symbol Connector:TestPoint
- added TP6: PCB_TX, TestPoint:TestPoint_Keystone_5015_Micro-Minature, symbol Connector:TestPoint
- added TP7: PCB_RX, TestPoint:TestPoint_Keystone_5015_Micro-Minature, symbol Connector:TestPoint
- added TP8: MotorM0, TestPoint:TestPoint_Keystone_5015_Micro-Minature, symbol Connector:TestPoint
- added TP9: MotorM1, TestPoint:TestPoint_Keystone_5015_Micro-Minature, symbol Connector:TestPoint
- A1: value Pololu_Breakout_DRV8825 -> DRV8825
- C11: renamed from C6; value 2.2uF -> 22uF; MPN 08056C225KAT2A -> C0805C226M8PACTU; Manufacturer (none) -> KEMET
- C2: renamed from C4; Manufacturer (none) -> TDK
- C7, C8, C9: footprint Capacitor_SMD:C_0603_1608Metric -> Capacitor_SMD:C_0805_2012Metric; MPN CGB1T3X6S0G104M022BB -> AS0805KKX7R9BB104; Manufacturer TDK -> Yageo
- J2: renamed from J1; value Header_02x02 -> Programmer; footprint Connector_PinHeader_1.00mm:PinHeader_2x02_P1.00mm_Vertical -> Connector_PinHeader_2.54mm:PinHeader_2x02_P2.54mm_Vertical
- J3: renamed from MotorConnector_Female1; value JST_1x6_Female -> MotorConnector; footprint Connector_JST:JST_EH_B02B-EH-A_1x06_P2.50mm_Vertical -> Connector_JST:JST_XH_B6B-XH-AM_1x06_P2.50mm_Vertical
- J4: renamed from Temp_Female1; value JST_1x2_Female -> TempSensor; footprint Connector_JST:JST_EH_B02B-EH-A_1x02_P2.50mm_Vertical -> Connector_JST:JST_XH_B2B-XH-AM_1x02_P2.50mm_Vertical
- J5: renamed from USB_B_Header1; value USB -> USB_B; symbol electrospinner-rescue:USB_B-Connector -> Connector:USB_B
- R7: renamed from R1; footprint Resistor_SMD:R_0603 -> Resistor_SMD:R_0805_2012Metric
- renumbered C2 to C1, C1 to C3, C3 to C5, L2 to L1, R3 to R1, R4 to R2, R7 to R4, U3 to U1, U1 to U2, U5 to U3
Connections:
- net labels added: A1, A2, B1, B2, MotorM0, MotorM1, MotorM2, ~MotorEN, ~MotorSLP
- net labels removed: 1A, 1B, 2A, 2B, BLK, BLU, GRN, MotorMS#, MotorMS1, MotorMS2, MotorMS3, MotorSLEEP, RED, WHT, YEL, ~MotorENABLE, ~MotorRESET, ~MotorSLEEP
- wire segments 171 -> 150
Other:
- note added: "BLACK"
- note added: "BLUE"
- note added: "GREEN"
- note added: "RED"
- note added: "WHITE"
- note added: "YELLOW"
- moved on the sheet: A1, C1, C3, C5, D1, D2, J2, J3, J4, J5, L1, R4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
