File: board/electrospinner-pcb/electrospinner.kicad_pcb (KiCad board)
At the start: 2 copper layers, 27 parts, among them J1 Header_02x02, SW1 ResetBTN, U1 FT230XS, U5 MSP430G2553IPW20

Commit message: Updates to rev5
Parts:
- removed Barrel_Jack1: BarrelJack, Connector_BarrelJack:BarrelJack_Horizontal
- removed C10: 0.1uF, Capacitor_SMD:C_0603_1608Metric
- removed L2: 1uH, Inductor_SMD:L_0805_2012Metric
- removed R3: 560k, Resistor_SMD:R_0805_2012Metric
- removed Temp_Female1: JST_1x2_Female, Connector_JST:JST_EH_B02B-EH-A_1x02_P2.50mm_Vertical
- removed U5: MSP430G2553IPW20, Package_SO:TSSOP-20_4.4x6.5mm_P0.65mm
- removed USB_B_Header1: USB_B_Header?, Connector_USB:USB_B_OST_USB-B1HSxx_Horizontal
- added C11: 22uF, Capacitor_SMD:C_0805_2012Metric, F.Cu at (190.5, 89.2)
- added J2: Programmer, Connector_PinHeader_2.54mm:PinHeader_2x02_P2.54mm_Vertical, F.Cu at (128.3, 58.4)
- added J3: MotorConnector, Connector_JST:JST_XH_B6B-XH-AM_1x06_P2.50mm_Vertical, F.Cu at (114.3, 59.7)
- added J4: TempSensor, Connector_JST:JST_XH_B2B-XH-AM_1x02_P2.50mm_Vertical, F.Cu at (165.1, 74.9)
- added J5: USB_B, Connector_USB:USB_B_OST_USB-B1HSxx_Horizontal, F.Cu at (113.0, 114.3)
- added L1: 1uH, Inductor_SMD:L_0805_2012Metric, F.Cu at (186.7, 86.7)
- added R1: 560k, Resistor_SMD:R_0805_2012Metric, F.Cu at (181.9, 91.4)
- added TP1: ~MotorRST, TestPoint:TestPoint_Keystone_5015_Micro-Minature, F.Cu at (160.0, 91.4)
- added TP10: MotorM2, TestPoint:TestPoint_Keystone_5015_Micro-Minature, F.Cu at (160.0, 94.0)
- added TP11: MotorSTEP, TestPoint:TestPoint_Keystone_5015_Micro-Minature, F.Cu at (160.0, 86.4)
- added TP2: ~MotorEN, TestPoint:TestPoint_Keystone_5015_Micro-Minature, F.Cu at (160.0, 101.6)
- added TP3: ~MotorSLP, TestPoint:TestPoint_Keystone_5015_Micro-Minature, F.Cu at (160.0, 88.9)
- added TP4: MotorDIR, TestPoint:TestPoint_Keystone_5015_Micro-Minature, F.Cu at (160.0, 83.8)
- added TP5: ~MotorFLT, TestPoint:TestPoint_Keystone_5015_Micro-Minature, F.Cu at (130.8, 86.4)
- added TP6: PCB_TX, TestPoint:TestPoint_Keystone_5015_Micro-Minature, F.Cu at (135.9, 54.6)
- added TP7: PCB_RX, TestPoint:TestPoint_Keystone_5015_Micro-Minature, F.Cu at (124.5, 104.1)
- added TP8: MotorM0, TestPoint:TestPoint_Keystone_5015_Micro-Minature, F.Cu at (160.0, 99.1)
- added TP9: MotorM1, TestPoint:TestPoint_Keystone_5015_Micro-Minature, F.Cu at (160.0, 96.5)
- added U2: FT230XS, Package_SO:SSOP-16_3.9x4.9mm_P0.635mm, F.Cu at (124.5, 111.8)
- added U3: MSP430G2553IPW20, Package_SO:TSSOP-20_4.4x6.5mm_P0.65mm, F.Cu at (149.9, 67.3)
- A1: value A4988_Breakout -> DRV8825
- C1: value 0.1uF -> 10uF
- C2: value 10uF -> 3.3uF
- C3: value 100uF -> 0.1uF; footprint Capacitor_SMD:CP_Elec_6.3x5.8 -> Capacitor_SMD:C_0805_2012Metric
- C4: value 3.3uF -> 0.1uF
- C5: value 0.1uF -> 100uF; footprint Capacitor_SMD:C_0603_1608Metric -> Capacitor_SMD:CP_Elec_6.3x5.8
- C6: value 2.2uF -> 0.1uF
- C7, C8, C9: footprint Capacitor_SMD:C_0603_1608Metric -> Capacitor_SMD:C_0805_2012Metric
- J1: value Header_02x02 -> 12Vin; footprint Connector_PinHeader_1.00mm:PinHeader_2x02_P1.00mm_Vertical -> Connector_BarrelJack:BarrelJack_CUI_PJ-063AH_Horizontal
- R2: value 100 -> 150k
- R4: value 150k -> 10k
- R7: value 10k -> 158
- U1: value FT230XS -> TPS62147; footprint Package_SO:SSOP-16_3.9x4.9mm_P0.635mm -> footprints:TPS62147RGXR
- moved J1 65.0 mm to (109.9, 94.6), turned to 270 degrees
- moved SW1 62.5 mm to (146.1, 54.6)
- moved R6 61.9 mm to (121.9, 123.2), turned to 90 degrees
- moved R5 60.4 mm to (124.5, 123.2), turned to 90 degrees
- moved A1 60.3 mm to (137.2, 83.8), turned to 0 degrees
- moved C2 57.5 mm to (180.3, 86.4), turned to 270 degrees
- moved D2 57.1 mm to (121.9, 119.4), turned to 90 degrees
- moved C8 55.8 mm to (129.5, 111.8), turned to 270 degrees
- moved D1 55.4 mm to (124.5, 119.4), turned to 270 degrees
- moved C4 53.6 mm to (188.5, 98.4)
- moved C5 52.1 mm to (132.1, 100.3), turned to 90 degrees
- moved C6 42.7 mm to (180.2, 105.6)
- moved C1 28.8 mm to (128.3, 116.8), turned to 180 degrees
- moved R2 27.4 mm to (186.7, 91.4)
- moved C3 26.2 mm to (137.2, 104.1), turned to 180 degrees
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Connections:
- A1 pad 10: /MOTOR_MS1 -> /MotorM0
- A1 pad 11: /MOTOR_MS2 -> /MotorM1
- A1 pad 12: /MOTOR_MS3 -> /MotorM2
- A1 pad 13: /~MOTOR_RESET -> /~MotorRST
- A1 pad 14: /~MOTOR_SLEEP -> /~MotorSLP
- A1 pad 15: /MOTOR_STEP -> /MotorSTEP
- A1 pad 16: /MOTOR_DIR -> /MotorDIR
- A1 pad 2: +3V3 -> /~MotorFLT
- A1 pad 3: /1B -> /A2
- A1 pad 4: /1A -> /A1
- A1 pad 5: /2A -> /B1
- A1 pad 6: /2B -> /B2
- A1 pad 9: /~MOTOR_ENABLE -> /~MotorEN
- C2 pad 1: +12V -> Net-(C2-Pad1)
- C4 pad 1: Net-(C4-Pad1) -> +12V
- C5 pad 1: +3V3 -> +12V
- J1 pad 1: /DVCC -> +12V
- J1 pad 2: /DVSS -> GNDD
- R2 pad 1: /~RST -> Net-(R1-Pad2)
- R2 pad 2: Net-(C10-Pad2) -> GNDD
- R4 pad 1: Net-(R3-Pad2) -> /~RST
- R7 pad 1: /~RST -> /Vo,temp
- U1 pad 1: /PCB_TX -> +12V
- U1 pad 10: Net-(U1-Pad10) -> GNDD
- U1 pad 11: /~RST -> +12V
- U1 pad 3: +3V3 -> GNDD
- U1 pad 4: /PCB_RX -> GNDD
- U1 pad 5: GNDD -> Net-(R1-Pad2)
- U1 pad 6: Net-(U1-Pad6) -> +3V3
- U1 pad 7: /~TXLED -> GNDD
- U1 pad 8: /D+ -> +12V
- U1 pad 9: /D- -> Net-(C2-Pad1)
Routing:
- net +3V3: track 88.7 -> 0.00 mm, vias 3 -> 0
- net GNDD: track 74.9 -> 0.00 mm
- net /~RST: track 33.1 -> 0.00 mm
- net /PCB_RX: track 24.1 -> 0.00 mm, vias 2 -> 0
- net /PCB_TX: track 23.8 -> 0.00 mm, vias 2 -> 0
- net /D-: track 19.7 -> 0.00 mm
- net /Vo,temp: track 17.8 -> 0.00 mm
- net +12V: track 16.6 -> 0.00 mm
- net /~RXLED: track 8.46 -> 0.00 mm
- net /D+: track 7.92 -> 0.00 mm
- net /~TXLED: track 7.74 -> 0.00 mm
- net /TEST: track 4.16 -> 0.00 mm
- net Net-(C10-Pad2): track 2.60 -> 0.00 mm
- net Net-(D2-Pad2): track 2.09 -> 0.00 mm
- net Net-(D1-Pad2): track 2.09 -> 0.00 mm
