File: board/electrospinner.sch (KiCad schematic (older format))
At the start: 42 parts, among them J1 12Vin, J2 Programmer, J3 MotorConnector, J4 TempSensorConnector, J5 USB_B, SW1 ResetBTN, U1 TPS62147, U2 FT230XS, U3 MSP430G2553IPW20

Commit message: Updates the BOM and layout for rev6
Parts:
- D1, D2, J2, J3, J4, J5, SW1: MPN (none) -> resource-center; Manufacturer (none) -> resource-center
- J1: MPN (none) -> resource-center; Manufacturer (none) -> resource-center; Status (none) -> resource-center
- L1: footprint Inductor_SMD:L_0805_2012Metric -> electrospinner:L_Coilcraft_XEL6030; MPN DFE201612PD-1R0M=P2 -> XEL6030-222MEC; Manufacturer (none) -> Coilcraft
- TP1, TP10, TP11, TP2, TP3, TP4, TP5, TP6, TP7, TP8, TP9: MPN (none) -> 5015; Manufacturer (none) -> Keystone Electronics
- U1, U3: Manufacturer (none) -> Texas Instruments
Changed lines of the file:
@@
 F 3 " ~" H 1250 4600 50  0001 C CNN
 F 4 "resource-center" H -350 -2150 50  0001 C CNN "Status"
+F 5 "resource-center" H 0   0   50  0001 C CNN "MPN"
+F 6 "resource-center" H 0   0   50  0001 C CNN "Manufacturer"
 	1    1100 4650
 	1    0    0    -1
@@
 F 3 "http://www.ti.com/lit/gpn/tps62147" H 1650 1900 50  0001 C CNN
 F 4 "TPS62147RGXR" H -700 50  50  0001 C CNN "MPN"
+F 5 "Texas Instruments" H 0   0   50  0001 C CNN "Manufacturer"
 	1    1650 1900
 	1    0    0    -1
@@
 F 0 "L1" V 2435 2200 50  0000 C CNN
 F 1 "2.2uH" V 2344 2200 50  0000 C CNN
-F 2 "Inductor_SMD:L_0805_2012Metric" H 2250 2200 50  0001 C CNN
-F 3 "https://www.mouser.com/datasheet/2/281/J(E)TE243A-9101-1324383.pdf" H 2250 2200 50  0001 C CNN
-F 4 "DFE201612PD-1R0M=P2" H -800 50  50  0001 C CNN "MPN"
+F 2 "electrospinner:L_Coilcraft_XEL6030" H 2250 2200 50  0001 C CNN
+F 3 "https://www.mouser.com/datasheet/2/597/xel6030-1359473.pdf" H 2250 2200 50  0001 C CNN
+F 4 "XEL6030-222MEC" H -800 50  50  0001 C CNN "MPN"
+F 5 "Coilcraft" H 0   0   50  0001 C CNN "Manufacturer"
 	1    2250 2200
 	0    -1   -1   0
@@
 F 3 "~" V 4100 4950 50  0001 C CNN
 F 4 "resource-center" H 950 -400 50  0001 C CNN "Status"
+F 5 "resource-center" H 0   0   50  0001 C CNN "MPN"
+F 6 "resource-center" H 0   0   50  0001 C CNN "Manufacturer"
 	1    4100 4950
 	1    0    0    -1
@@
 F 3 "~" V 4100 5050 50  0001 C CNN
 F 4 "resource-center" H 950 -400 50  0001 C CNN "Status"
+F 5 "resource-center" H 0   0   50  0001 C CNN "MPN"
+F 6 "resource-center" H 0   0   50  0001 C CNN "Manufacturer"
 	1    4100 5050
 	1    0    0    -1
@@
 F 3 "~" H 9400 4550 50  0001 C CNN
 F 4 "resource-center" H 2200 -850 50  0001 C CNN "Status"
+F 5 "resource-center" H 0   0   50  0001 C CNN "MPN"
+F 6 "resource-center" H 0   0   50  0001 C CNN "Manufacturer"
 	1    9400 4550
 	1    0    0    -1
@@
 F 3 "~" H 5800 1350 50  0001 C CNN
 F 4 "resource-center" H -4200 -1050 50  0001 C CNN "Status"
+F 5 "resource-center" H 0   0   50  0001 C CNN "MPN"
+F 6 "resource-center" H 0   0   50  0001 C CNN "Manufacturer"
 	1    5800 1350
 	1    0    0    -1
@@
 F 3 "http://www.ti.com/lit/ds/symlink/msp430g2553.pdf" H 6650 2450 50  0001 C CNN
 F 4 "MSP430G2553IPW20" H 0   0   50  0001 C CNN "MPN"
+F 5 "Texas Instruments" H 0   0   50  0001 C CNN "Manufacturer"
 	1    6700 2450
 	1    0    0    -1
@@
 F 3 "~" H 3250 1550 50  0001 C CNN
 F 4 "resource-center" H -1200 -400 50  0001 C CNN "Status"
+F 5 "resource-center" H 0   0   50  0001 C CNN "MPN"
+F 6 "resource-center" H 0   0   50  0001 C CNN "Manufacturer"
 	1    3250 1350
 	0    1    -1   0
@@
 F 1 "~MotorRST" V 4550 2700 50  0000 C CNN
 F 2 "TestPoint:TestPoint_Keystone_5015_Micro-Minature" H 4750 2150 50  0001 C CNN
-F 3 "~" H 4750 2150 50  0001 C CNN
+F 3 "https://www.mouser.com/datasheet/2/215/015-744075.pdf" H 4750 2150 50  0001 C CNN
+F 4 "5015 " H 0   0   50  0001 C CNN "MPN"
+F 5 "Keystone Electronics" H 0   0   50  0001 C CNN "Manufacturer"
 	1    4550 2150
 	0    -1   -1   0
@@
 F 3 "~" H 10700 1950 50  0001 C CNN
 F 4 "resource-center" H 1350 950 50  0001 C CNN "Status"
+F 5 "resource-center" H 0   0   50  0001 C CNN "MPN"
+F 6 "resource-center" H 0   0   50  0001 C CNN "Manufacturer"
 	1    10700 1950
 	1    0    0    -1
@@
 F 1 "~MotorEN" V 4550 2800 50  0000 C CNN
 F 2 "TestPoint:TestPoint_Keystone_5015_Micro-Minature" H 4750 2250 50  0001 C CNN
-F 3 "~" H 4750 2250 50  0001 C CNN
+F 3 "https://www.mouser.com/datasheet/2/215/015-744075.pdf" H 4750 2250 50  0001 C CNN
+F 4 "5015 " H 0   0   50  0001 C CNN "MPN"
+F 5 "Keystone Electronics" H 0   0   50  0001 C CNN "Manufacturer"
 	1    4550 2250
 	0    -1   -1   0
@@
 F 1 "PCB_TX" V 8900 2550 50  0000 L CNN
 F 2 "TestPoint:TestPoint_Keystone_5015_Micro-Minature" H 9100 2150 50  0001 C CNN
-F 3 "~" H 9100 2150 50  0001 C CNN
+F 3 "https://www.mouser.com/datasheet/2/215/015-744075.pdf" H 9100 2150 50  0001 C CNN
+F 4 "5015 " H 0   0   50  0001 C CNN "MPN"
+F 5 "Keystone Electronics" H 0   0   50  0001 C CNN "Manufacturer"
 	1    8900 2150
 	0    1    1    0
@@
 F 1 "PCB_RX" V 8900 2650 50  0000 L CNN
 F 2 "TestPoint:TestPoint_Keystone_5015_Micro-Minature" H 9100 2250 50  0001 C CNN
-F 3 "~" H 9100 2250 50  0001 C CNN
+F 3 "https://www.mouser.com/datasheet/2/215/015-744075.pdf" H 9100 2250 50  0001 C CNN
+F 4 "5015 " H 0   0   50  0001 C CNN "MPN"
+F 5 "Keystone Electronics" H 0   0   50  0001 C CNN "Manufacturer"
 	1    8900 2250
 	0    1    1    0
@@
 F 1 "MotorM0" V 8900 2750 50  0000 L CNN
 F 2 "TestPoint:TestPoint_Keystone_5015_Micro-Minature" H 9100 2350 50  0001 C CNN
-F 3 "~" H 9100 2350 50  0001 C CNN
+F 3 "https://www.mouser.com/datasheet/2/215/015-744075.pdf" H 9100 2350 50  0001 C CNN
+F 4 "5015 " H 0   0   50  0001 C CNN "MPN"
+F 5 "Keystone Electronics" H 0   0   50  0001 C CNN "Manufacturer"
 	1    8900 2350
 	0    1    1    0
@@
 F 1 "MotorM1" V 8900 2850 50  0000 L CNN
 F 2 "TestPoint:TestPoint_Keystone_5015_Micro-Minature" H 9100 2450 50  0001 C CNN
-F 3 "~" H 9100 2450 50  0001 C CNN
+F 3 "https://www.mouser.com/datasheet/2/215/015-744075.pdf" H 9100 2450 50  0001 C CNN
+F 4 "5015 " H 0   0   50  0001 C CNN "MPN"
+F 5 "Keystone Electronics" H 0   0   50  0001 C CNN "Manufacturer"
 	1    8900 2450
 	0    1    1    0
@@
 F 1 "MotorM2" V 8900 2950 50  0000 L CNN
 F 2 "TestPoint:TestPoint_Keystone_5015_Micro-Minature" H 9100 2550 50  0001 C CNN
-F 3 "~" H 9100 2550 50  0001 C CNN
+F 3 "https://www.mouser.com/datasheet/2/215/015-744075.pdf" H 9100 2550 50  0001 C CNN
+F 4 "5015 " H 0   0   50  0001 C CNN "MPN"
+F 5 "Keystone Electronics" H 0   0   50  0001 C CNN "Manufacturer"
 	1    8900 2550
 	0    1    1    0
@@
 F 1 "~MotorSLP" V 4550 2900 50  0000 C CNN
 F 2 "TestPoint:TestPoint_Keystone_5015_Micro-Minature" H 4750 2350 50  0001 C CNN
-F 3 "~" H 4750 2350 50  0001 C CNN
+F 3 "https://www.mouser.com/datasheet/2/215/015-744075.pdf" H 4750 2350 50  0001 C CNN
+F 4 "5015 " H 0   0   50  0001 C CNN "MPN"
+F 5 "Keystone Electronics" H 0   0   50  0001 C CNN "Manufacturer"
 	1    4550 2350
 	0    -1   -1   0
@@
 F 1 "MotorDIR" V 4550 3000 50  0000 C CNN
 F 2 "TestPoint:TestPoint_Keystone_5015_Micro-Minature" H 4750 2450 50  0001 C CNN
-F 3 "~" H 4750 2450 50  0001 C CNN
+F 3 "https://www.mouser.com/datasheet/2/215/015-744075.pdf" H 4750 2450 50  0001 C CNN
+F 4 "5015 " H 0   0   50  0001 C CNN "MPN"
+F 5 "Keystone Electronics" H 0   0   50  0001 C CNN "Manufacturer"
 	1    4550 2450
 	0    -1   -1   0
@@
 F 1 "~MotorFLT" V 4550 3100 50  0000 C CNN
 F 2 "TestPoint:TestPoint_Keystone_5015_Micro-Minature" H 4750 2550 50  0001 C CNN
-F 3 "~" H 4750 2550 50  0001 C CNN
+F 3 "https://www.mouser.com/datasheet/2/215/015-744075.pdf" H 4750 2550 50  0001 C CNN
+F 4 "5015 " H 0   0   50  0001 C CNN "MPN"
+F 5 "Keystone Electronics" H 0   0   50  0001 C CNN "Manufacturer"
 	1    4550 2550
 	0    -1   -1   0
@@
 F 1 "MotorSTEP" V 8900 3050 50  0000 L CNN
 F 2 "TestPoint:TestPoint_Keystone_5015_Micro-Minature" H 9100 2650 50  0001 C CNN
-F 3 "~" H 9100 2650 50  0001 C CNN
+F 3 "https://www.mouser.com/datasheet/2/215/015-744075.pdf" H 9100 2650 50  0001 C CNN
+F 4 "5015 " H 0   0   50  0001 C CNN "MPN"
+F 5 "Keystone Electronics" H 0   0   50  0001 C CNN "Manufacturer"
 	1    8900 2650
 	0    1    1    0
@@
 F 2 "Connector_BarrelJack:BarrelJack_CUI_PJ-063AH_Horizontal" H 950 1010 50  0001 C CNN
 F 3 "~" H 950 1010 50  0001 C CNN
+F 4 "resource-center" H 0   0   50  0001 C CNN "MPN"
+F 5 "resource-center" H 0   0   50  0001 C CNN "Manufacturer"
+F 6 "resource-center" H 0   0   50  0001 C CNN "Status"
 	1    900  1050
 	1    0    0    -1

Commit message: Updates for rev7
Adds project specific symbol and footprint libraries
Adds thermocouple_amplifier datasheet
Parts:
- added C13: 0.1uF, Capacitor_SMD:C_0805_2012Metric, symbol Device:C_Small
- added D3: LedRED, LED_SMD:LED_0603_1608Metric, symbol electrospinner-rescue:LED_Small-Device-electrospinner-rescue
- added D5: LedGRN, LED_SMD:LED_0603_1608Metric, symbol electrospinner-rescue:LED_Small-Device-electrospinner-rescue
- added J6: FanConnector, Connector_JST:JST_XH_B2B-XH-AM_1x02_P2.50mm_Vertical, symbol Connector:Conn_01x02_Female
- added Q1: 2N7000, Package_TO_SOT_THT:TO-92_Inline, symbol Transistor_FET:2N7000
- added R11, R9: 390, Resistor_SMD:R_0805_2012Metric, symbol electrospinner-rescue:R_Small_US-Device-electrospinner-rescue-electrospinner-re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
- added R3: 75k, Resistor_SMD:R_0805_2012Metric, symbol Device:R_Small_US
- added R8: 1M, Resistor_SMD:R_0805_2012Metric, symbol Device:R_Small_US
- added U4: AD8495, Package_SO:MSOP-8_3x3mm_P0.65mm, symbol Sensor_Temperature:AD8495
- C1, C11, C12: symbol electrospinner-rescue:C_Small-Device-electrospinner-rescue -> electrospinner-rescue:C_Small-Device-electrospinner-rescue-electrospinner-rescue
- C10: value 10uF -> 1uF; footprint Capacitor_SMD:C_0805_2012Metric -> Capacitor_SMD:CP_Elec_4x5.4; MPN C0805X106K8RACAUTO -> EXV105M050A9BAA
- C2: symbol electrospinner-rescue:C_Small-Device -> electrospinner-rescue:C_Small-Device-electrospinner-rescue-electrospinner-rescue
- D1: value RXLED -> LedRX; symbol electrospinner-rescue:LED_Small-Device -> electrospinner-rescue:LED_Small-Device-electrospinner-rescue
- D2: value TXLED -> LedTX; symbol electrospinner-rescue:LED_Small-Device -> electrospinner-rescue:LED_Small-Device-electrospinner-rescue
- J2: symbol electrospinner-rescue:Conn_02x02_Counter_Clockwise-Connector_Generic -> electrospinner-rescue:Conn_02x02_Counter_Clockwise-Connector_Generic-electrospinner-rescue
- J3: symbol electrospinner-rescue:Conn_01x06_Female-Connector -> electrospinner-rescue:Conn_01x06_Female-Connector-electrospinner-rescue
- J4: symbol electrospinner-rescue:Conn_01x02_Female-Connector -> electrospinner-rescue:Conn_01x02_Female-Connector-electrospinner-rescue
- L1: footprint electrospinner:L_Coilcraft_XEL6030 -> libs:L_Coilcraft_XEL6030; symbol electrospinner-rescue:L_Small-Device-electrospinner-rescue -> electrospinner-rescue:L_Small-Device-electrospinner-rescue-electrospinner-rescue
- R1, R2: symbol electrospinner-rescue:R_Small_US-Device-electrospinner-rescue -> electrospinner-rescue:R_Small_US-Device-electrospinner-rescue-electrospinner-rescue
- R4, R5, R6: symbol electrospinner-rescue:R_Small_US-Device -> electrospinner-rescue:R_Small_US-Device-electrospinner-rescue-electrospinner-rescue
- R7: value 158 -> 75k; MPN CR0603-FX-1580ELF -> ERJ-6RBD7502V; Manufacturer Bourns -> Panasonic
- SW1: symbol electrospinner-rescue:SW_Push-Switch -> electrospinner-rescue:SW_Push-Switch-electrospinner-rescue
- U1: footprint footprints:TPS62147RGXR -> libs:TPS62147RGXR; symbol electrospinner-rescue:TPS62147-Regulator_Switching-electrospinner-rescue-electrospinner-rescue -> electrospinner-rescue:TPS62147-Regulator_Switching-electrospinner-rescue-electrospinner-rescue-electrospinner-rescue
- U2: symbol electrospinner-rescue:FT230XS-Interface_USB -> electrospinner-rescue:FT230XS-Interface_USB-electrospinner-rescue
- U3: symbol electrospinner-rescue:MSP430G2553IPW20-MCU_Texas_MSP430-electrospinner-rescue -> electrospinner-rescue:MSP430G2553IPW20-MCU_Texas_MSP430-electrospinner-rescue-electrospinner-rescue
Connections:
- net +12V: now also Q1.3 (D); no longer A1.8 (VMOT), C1.1, C4.1, U1.1 (VIN), U1.8 (EN)
- net +3V3: now also C4.1; no longer C10.1, C9.1, J4.1 (Pin_1), U2.12 (VCC), U2.3 (VCCIO), U3.1 (DVCC)
- net MotorM0: now also U3.13 (P2.5/TA1.2); no longer U3.5 (CAOUT/VREF-/VeREF-/CA3/A3/P1.3)
- net MotorM1: now also U3.19 (P2.6/XIN/TA0.1); no longer U3.6 (TCK/SMCLK/UCB0STE/UCA0CLK/VREF+/VeREF+/CA4/A4/P1.4)
- net MotorM2: now also U3.18 (P2.7/XOUT); no longer U3.7 (TMS/UCB0CLK/UCA0STE/TA0.0/CA5/A5/P1.5)
- net Vo,temp: now also U4.5 (SENSE), U4.6; no longer J4.2 (Pin_2), R7.1
- net LedGRN: now reaches U3.15 (TDO/TDI/UCB0SIMO/UCB0SDA/CAOUT/CA7/A7/P1.7)
- net LedGRN: now also U3.6 (TCK/SMCLK/UCB0STE/UCA0CLK/VREF+/VeREF+/CA4/A4/P1.4), D5.2 (A)
- net GNDD renamed GND
- net GND: now also C9.1, C13.2, J6.2 (Pin_2), R11.1, R8.1, R9.1, U4.2 (REF), U4.3 (-Vs); no longer C10.2, C3.2, C4.2, C5.2, C6.2, C7.2, C8.2, C9.2, R7.2
- net ~RXLED renamed ~LedRX
- net ~TXLED renamed ~LedTX
- new net: C6.2, U3.1 (DVCC)
- new net: J4.1 (Pin_1), R3.1, R8.2
- new net: J4.2 (Pin_2), R7.1
- new net: C1.1, C3.2, U1.1 (VIN), U1.8 (EN)
- new net: C7.2, U2.12 (VCC)
- new net: C8.2, U2.3 (VCCIO)
- new net: A1.8 (VMOT), C5.2
- new net: C10.1, C9.2, R3.2, U4.1 (-IN)
- new net: C4.2, U4.7 (+Vs)
- new net: C10.2, C13.1, R7.2, U4.8 (+IN)
- new net: D3.1 (K), R9.2
- new net: D5.1 (K), R11.2
- new net: J6.1 (Pin_1), Q1.1 (S)
- new net FAN: Q1.2 (G), U3.7 (TMS/UCB0CLK/UCA0STE/TA0.0/CA5/A5/P1.5)
- new net LedRED: D3.2 (A), U3.5 (CAOUT/VREF-/VeREF-/CA3/A3/P1.3)
- no-connect marks 12 -> 8
Other:
- note added: "Buck Converter 12V to 3V3"
- note added: "Fan Control"
- note added: "Termperature Sensor"
- note added: "Voltage Regulation"
- note removed: "Buck Converter"
- note removed: "Temperature Sensing Circuit"
- moved on the sheet: A1, C1, C11, C12, C2, C5, C6, C7, C8, D1, D2, J1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
